File: examples/pcb_led_board/artifacts/pcb_led_board.kicad_pcb (KiCad board)
At the start: 2 copper layers, 32 x 18 mm, 5 parts, among them J1 Two-pin connector

Commit message: Keep board holes generic
Parts:
- ? (x2): footprint MountingHole_NPTH -> BoardHole_NPTH
Changed lines of the file:
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@@
   (net 2 "LED_A")
   (net 3 "GND")
-  (footprint "MountingHole_NPTH"
+  (footprint "BoardHole_NPTH"
     (layer "F.Cu")
     (at 3 3)
@@
     )
   )
-  (footprint "MountingHole_NPTH"
+  (footprint "BoardHole_NPTH"
     (layer "F.Cu")
     (at 29 15)
