File: tests/fixtures/kicad_flat_resistor.kicad_pcb (KiCad board)
At the start: 2 copper layers, 50 x 30 mm, 2 parts

Commit message: Keep board holes generic
Parts:
- ?: footprint MountingHole_NPTH -> BoardHole_NPTH
Changed lines of the file:
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@@
   (net 1 "LEFT")
   (net 2 "RIGHT")
-  (footprint "MountingHole_NPTH"
+  (footprint "BoardHole_NPTH"
     (layer "F.Cu")
     (at 3 3)
