File: tests/fixtures/kicad_flat_resistor.kicad_pcb (KiCad board)
At the start: 2 copper layers, 50 x 30 mm, 2 parts

Commit message: Correct KiCad rotation convention
Parts:
- turned R1 to 270 degrees
Changed lines of the file:
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@@
   (footprint "R_0603_1608Metric"
     (layer "F.Cu")
-    (at 25 15 90)
+    (at 25 15 270)
     (property "Reference" "R1"
       (at 0 -1.5 0)
@@
     (attr smd)
     (pad "1" smd roundrect
-      (at -0.75 0 90)
+      (at -0.75 0 270)
       (size 0.8 0.95)
       (layers "F.Cu" "F.Paste" "F.Mask")
@@
     )
     (pad "2" smd roundrect
-      (at 0.75 0 90)
+      (at 0.75 0 270)
       (size 0.8 0.95)
       (layers "F.Cu" "F.Paste" "F.Mask")
