File: examples/stm32_usb_buck/artifacts/stm32_usb_buck.kicad_pcb (KiCad board)
At the start: 4 copper layers, 90 x 58 mm, 28 parts, among them J2 SWD 10-pin, J3 GPIO 1x4, SW1 BOOT0, U1 STM32F405RGT6, Y1 8 MHz

Commit message: Add explicit Board resolution
Routing:
- net STATUS_LED: track 0.00 -> 39.1 mm
Changed lines of the file:
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@@
     (net 41)
+  )
+  (segment
+    (start 43.2 34.25)
+    (end 44.15 34.25)
+    (width 0.2)
+    (layer "F.Cu")
+    (net 38)
+  )
+  (segment
+    (start 44.15 34.25)
+    (end 44.15 51.9)
+    (width 0.2)
+    (layer "F.Cu")
+    (net 38)
+  )
+  (segment
+    (start 44.15 51.9)
+    (end 45.1 51.9)
+    (width 0.2)
+    (layer "F.Cu")
+    (net 38)
+  )
+  (segment
+    (start 45.1 51.9)
+    (end 62.75 51.9)
+    (width 0.2)
+    (layer "F.Cu")
+    (net 38)
+  )
+  (segment
+    (start 62.75 51.9)
+    (end 62.75 50)
+    (width 0.2)
+    (layer "F.Cu")
+    (net 38)
   )
   (via
